Commit message: dynamic port added

File: urdf/diffbot.ros2_control.xacro (robot description, xacro)
@@ -1,5 +1,5 @@
 <?xml version="1.0"?>
 <robot xmlns:xacro="http://www.ros.org/wiki/xacro">
-  <xacro:macro name="diffbot_ros2_control" params="name prefix">
+  <xacro:macro name="diffbot_ros2_control" params="name prefix device:=/dev/ttyACM1 baud_rate:=57600">
     <ros2_control name="${name}" type="system">
       <hardware>
@@ -8,6 +8,6 @@
         <param name="right_wheel_name">${prefix}right_wheel_joint</param>
         <param name="loop_rate">30</param>
-        <param name="device">/dev/ttyACM0</param>
-        <param name="baud_rate">57600</param>
+        <param name="device">${device}</param>
+        <param name="baud_rate">${baud_rate}</param>
         <param name="timeout_ms">1000</param>
         <param name="enc_counts_per_rev">3436</param>
